File: input_power.kicad_sch (KiCad schematic)
At the start: 0 parts

Commit message: input power update
Parts:
- added C1: 6800u, symbol Device:C_Polarized
- added C2: 100n, symbol Device:C
- added D1: GBU8B, Diode_THT:Diode_Bridge_Vishay_GBU, symbol Diode_Bridge:GBU8B
- added F1: Fuse, symbol Device:Fuse
- added L, L_pierwotne_trafo, L_wtórne_trafo (x2), N, N_pierwotne_trafo: Conn_01x01_Pin, symbol Connector:Conn_01x01_Pin
- added RV1: Varistor, symbol Device:Varistor
Connections:
- new net: F1.2, L_pierwotne_trafo.1 (Pin_1), RV1.1
- new net: D1.2, L_wtórne_trafo.1 (Pin_1)
- new net: D1.3, L_wtórne_trafo.1 (Pin_1)
- new net GND: C1.2, C2.2, D1.4 (-)
- new net L: F1.1, L.1 (Pin_1)
- new net N: N.1 (Pin_1), N_pierwotne_trafo.1 (Pin_1), RV1.2
- new net Vin_32v: C1.1, C2.1, D1.1 (+)
