File: digital_power.kicad_sch (KiCad schematic)
At the start: 13 parts, among them U3 MC34063AD, U4 LM78L05_TO92

Commit message: zmiana sekcji zasilania digital oraz drivera
Parts:
- removed C11: 220p, symbol Device:C
- removed C12: 100p, symbol Device:C
- removed U4: LM78L05_TO92, Package_TO_SOT_THT:TO-92_Inline, symbol Regulator_Linear:LM78L05_TO92
- added C11, C12: 10u, symbol Device:C_Polarized
- added U5: NCP1117-3.3_SOT223, Package_TO_SOT_SMD:SOT-223-3_TabPin2, symbol Regulator_Linear:NCP1117-3.3_SOT223
- C10: value 330u -> 180u
- L2: value 220u -> 100u
- R5: value 7k -> 3.8k
Connections:
- net GND: now also C11.2, C12.2, U5.1 (GND)
- net Vout_10v: no longer names the net of C10.1, C9.1, L2.2, R5.2
- net Vout_10v: now also C12.1, U5.3 (VI)
- new net 3.3V: C11.1, U5.2 (VO)
Other:
- moved on the sheet: C10, C9

Commit message: dodanie testpointów, diody tvs, rezystora pomiarowego
Parts:
- added dodatkowe_3.3V_+, dodatkowe_3.3V_-, dodatkowe_6v: Conn_01x01_Pin, symbol Connector:Conn_01x01_Pin
Connections:
- net 3.3V: now also dodatkowe_3.3V_+.1 (Pin_1)
- net GND: now also dodatkowe_3.3V_-.1 (Pin_1)
- net at C10.1, C12.1, C9.1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: now also dodatkowe_6v.1 (Pin_1)

Commit message: dodanie footprintów do main buck (jeszcze driver i razystor bramek) poprawiony pinout LDI75L12UA, dodane footprinty do digital power
Parts:
- C10: footprint (none) -> Capacitor_SMD:CP_Elec_6.3x7.7
- C11, C12: footprint (none) -> Capacitor_SMD:CP_Elec_4x5.8
- C7: footprint (none) -> Capacitor_THT:CP_Radial_D10.0mm_P5.00mm
- C8, C9: footprint (none) -> Capacitor_SMD:C_0805_2012Metric_Pad1.18x1.45mm_HandSolder
- L2: footprint (none) -> Inductor_THT:L_Radial_D12.5mm_P7.00mm_Fastron_09HCP
- R3, R4, R5: footprint (none) -> Resistor_SMD:R_0805_2012Metric_Pad1.20x1.40mm_HandSolder
- dodatkowe_3.3V_+, dodatkowe_3.3V_-, dodatkowe_6v: footprint (none) -> Connector_PinHeader_2.54mm:PinHeader_1x01_P2.54mm_Vertical
Changed lines of the file:
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@@
 			)
 		)
-		(property "Footprint" ""
+		(property "Footprint" "Connector_PinHeader_2.54mm:PinHeader_1x01_P2.54mm_Vertical"
 			(at 143.51 81.28 0)
 			(hide yes)
@@
 			)
 		)
-		(property "Footprint" ""
+		(property "Footprint" "Resistor_SMD:R_0805_2012Metric_Pad1.20x1.40mm_HandSolder"
 			(at 104.14 94.488 90)
 			(hide yes)
@@
 			)
 		)
-		(property "Footprint" ""
+		(property "Footprint" "Capacitor_THT:CP_Radial_D10.0mm_P5.00mm"
 			(at 60.6552 66.04 0)
 			(hide yes)
@@
 			)
 		)
-		(property "Footprint" ""
+		(property "Footprint" "Capacitor_SMD:CP_Elec_4x5.8"
 			(at 150.8252 105.41 0)
 			(hide yes)
@@
 			)
 		)
-		(property "Footprint" ""
+		(property "Footprint" "Capacitor_SMD:C_0805_2012Metric_Pad1.18x1.45mm_HandSolder"
 			(at 124.1552 100.33 0)
 			(hide yes)
@@
 			)
 		)
-		(property "Footprint" ""
+		(property "Footprint" "Connector_PinHeader_2.54mm:PinHeader_1x01_P2.54mm_Vertical"
 			(at 176.53 114.3 0)
 			(hide yes)
@@
 			)
 		)
-		(property "Footprint" ""
+		(property "Footprint" "Capacitor_SMD:C_0805_2012Metric_Pad1.18x1.45mm_HandSolder"
 			(at 84.7852 77.47 0)
 			(hide yes)
@@
 			)
 		)
-		(property "Footprint" ""
+		(property "Footprint" "Inductor_THT:L_Radial_D12.5mm_P7.00mm_Fastron_09HCP"
 			(at 119.38 82.55 0)
 			(hide yes)
@@
 			)
 		)
-		(property "Footprint" ""
+		(property "Footprint" "Connector_PinHeader_2.54mm:PinHeader_1x01_P2.54mm_Vertical"
 			(at 177.8 85.09 0)
 			(hide yes)
@@
 			)
 		)
-		(property "Footprint" ""
+		(property "Footprint" "Capacitor_SMD:CP_Elec_6.3x7.7"
 			(at 135.5852 101.6 0)
 			(hide yes)
@@
 			)
 		)
-		(property "Footprint" ""
+		(property "Footprint" "Capacitor_SMD:CP_Elec_4x5.8"
 			(at 173.6852 102.87 0)
 			(hide yes)
@@
 			)
 		)
-		(property "Footprint" ""
+		(property "Footprint" "Resistor_SMD:R_0805_2012Metric_Pad1.20x1.40mm_HandSolder"
 			(at 92.71 94.488 90)
 			(hide yes)
@@
 			)
 		)
-		(property "Footprint" ""
+		(property "Footprint" "Resistor_SMD:R_0805_2012Metric_Pad1.20x1.40mm_HandSolder"
 			(at 100.33 47.498 90)
 			(hide yes)

Commit message: Dodanie brakującego połączenia do przycisków enkoderów
Parts:
- renumbered dodatkowe_3.3V_+ to dodatkowe_3.3V_+1, dodatkowe_3.3V_- to dodatkowe_3.3V_-1, dodatkowe_6v to dodatkowe_6v1
Changed lines of the file:
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@@
 		(dnp no)
 		(fields_autoplaced yes)
-		(property "Reference" "dodatkowe_6v"
+		(property "Reference" "dodatkowe_6v1"
 			(at 144.78 80.6449 90)
 			(show_name no)
@@
 			(project "zasilacz_projekt_kompetencyjny"
 				(path "/e9ad3936-200e-4b7c-85fb-533ca6ea54fd/38eb48c3-6dca-4780-b12d-acca55a9d974"
-					(reference "dodatkowe_6v")
+					(reference "dodatkowe_6v1")
 					(unit 1)
 				)
@@
 		(dnp no)
 		(fields_autoplaced yes)
-		(property "Reference" "dodatkowe_3.3V_-"
+		(property "Reference" "dodatkowe_3.3V_-1"
 			(at 177.8 112.3949 90)
 			(show_name no)
@@
 			(project "zasilacz_projekt_kompetencyjny"
 				(path "/e9ad3936-200e-4b7c-85fb-533ca6ea54fd/38eb48c3-6dca-4780-b12d-acca55a9d974"
-					(reference "dodatkowe_3.3V_-")
+					(reference "dodatkowe_3.3V_-1")
 					(unit 1)
 				)
@@
 		(dnp no)
 		(fields_autoplaced yes)
-		(property "Reference" "dodatkowe_3.3V_+"
+		(property "Reference" "dodatkowe_3.3V_+1"
 			(at 179.07 84.4549 90)
 			(show_name no)
@@
 			(project "zasilacz_projekt_kompetencyjny"
 				(path "/e9ad3936-200e-4b7c-85fb-533ca6ea54fd/38eb48c3-6dca-4780-b12d-acca55a9d974"
-					(reference "dodatkowe_3.3V_+")
-					(unit 1)
-				)
+					(reference "dodatkowe_3.3V_+1")
+					(unit 1)
+				)

Commit message: walidacja schematu, dodanie footprintu do drivera, ERC
Changed lines of the file:
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@@
+	)
+	(junction
+		(at 147.32 92.71)
+		(diameter 0)
+		(color 0 0 0 0)
 	)
 	(junction
@@
 	)
 	(junction
+		(at 88.9 58.42)
+		(diameter 0)
+		(color 0 0 0 0)
+	)
+	(junction
 		(at 113.03 58.42)
 		(diameter 0)
@@
 	)
 	(junction
+		(at 54.61 58.42)
+		(diameter 0)
+		(color 0 0 0 0)
+	)
+	(junction
 		(at 161.29 106.68)
 		(diameter 0)
@@
 		(color 0 0 0 0)
 	)
-	(junction
-		(at 88.9 58.42)
-		(diameter 0)
-		(color 0 0 0 0)
-	)
 	(wire
 		(pts
@@
 	(wire
 		(pts
+			(xy 54.61 58.42) (xy 59.69 58.42)
+		)
+		(stroke
+			(width 0)
+			(type default)
+		)
+	)
+	(wire
+		(pts
 			(xy 111.76 63.5) (xy 116.84 63.5)
 		)
@@
 	(wire
 		(pts
+			(xy 147.32 92.71) (xy 149.86 92.71)
+		)
+		(stroke
+			(width 0)
+			(type default)
+		)
+	)
+	(wire
+		(pts
 			(xy 96.52 92.71) (xy 97.79 92.71)
 		)
@@
 	(wire
 		(pts
-			(xy 50.8 58.42) (xy 59.69 58.42)
+			(xy 50.8 58.42) (xy 54.61 58.42)
 		)
 		(stroke
@@
 	(wire
 		(pts
+			(xy 88.9 58.42) (xy 91.44 58.42)
+		)
+		(stroke
+			(width 0)
+			(type default)
+		)
+	)
+	(wire
+		(pts
 			(xy 88.9 92.71) (xy 85.09 92.71)
 		)
@@
 	(wire
 		(pts
-			(xy 143.51 92.71) (xy 149.86 92.71)
-		)
-		(stroke
-			(width 0)
-			(type default)
-		)
-	)
-	(wire
-		(pts
-			(xy 88.9 58.42) (xy 91.44 58.42)
+			(xy 143.51 92.71) (xy 147.32 92.71)
 		)
 		(stroke
@@
 				)
 				(justify left)
+			)
+		)
+	)
+	(symbol
+		(lib_id "power:PWR_FLAG")
+		(at 54.61 58.42 0)
+		(unit 1)
+		(body_style 1)
+		(exclude_from_sim no)
+		(in_bom yes)
+		(on_board yes)
+		(in_pos_files yes)
+		(dnp no)
+		(fields_autoplaced yes)
+		(property "Reference" "#FLG01"
+			(at 54.61 56.515 0)
+			(hide yes)
+			(show_name no)
+			(do_not_autoplace no)
+			(effects
+				(font
+					(size 1.27 1.27)
+				)
+			)
+		)
+		(property "Value" "PWR_FLAG"
+			(at 54.61 53.34 0)
+			(show_name no)
+			(do_not_autoplace no)
+			(effects
+				(font
+					(size 1.27 1.27)
+				)
+			)
+		)
+		(property "Footprint" ""
+			(at 54.61 58.42 0)
+			(hide yes)
+			(show_name no)
+			(do_not_autoplace no)
+			(effects
+				(font
+					(size 1.27 1.27)
+				)
+			)
+		)
+		(property "Datasheet" ""
+			(at 54.61 58.42 0)
+			(hide yes)
+			(show_name no)
+			(do_not_autoplace no)
+			(effects
+				(font
+					(size 1.27 1.27)
+				)
+			)
+		)
+		(property "Description" "Special symbol for telling ERC where power comes from"
+			(at 54.61 58.42 0)
+			(hide yes)
+			(show_name no)
+			(do_not_autoplace no)
+			(effects
+				(font
+					(size 1.27 1.27)
+				)
+			)
+		)
+		(pin "1"
+		)
+		(instances
+			(project "zasilacz_projekt_kompetencyjny"
+				(path "/e9ad3936-200e-4b7c-85fb-533ca6ea54fd/38eb48c3-6dca-4780-b12d-acca55a9d974"
+					(reference "#FLG01")
+					(unit 1)
+				)
 			)
 		)
@@
 					(unit 1)
 				)
+			)
+		)
+	)
+	(symbol
+		(lib_id "power:PWR_FLAG")
+		(at 147.32 92.71 0)
+		(unit 1)
+		(body_style 1)
+		(exclude_from_sim no)
+		(in_bom yes)
+		(on_board yes)
+		(in_pos_files yes)
+		(dnp no)
+		(fields_autoplaced yes)
+		(property "Reference" "#FLG02"
+			(at 147.32 90.805 0)
+			(hide yes)
+			(show_name no)
+			(do_not_autoplace no)
+			(effects
+				(font
+					(size 1.27 1.27)
+				)
+			)
+		)
+		(property "Value" "PWR_FLAG"
+			(at 147.32 87.63 0)
+			(show_name no)
+			(do_not_autoplace no)
+			(effects
+				(font
+					(size 1.27 1.27)
+				)
+			)
+		)
+		(property "Footprint" ""
+			(at 147.32 92.71 0)
+			(hide yes)
+			(show_name no)
+			(do_not_autoplace no)
+			(effects
+				(font
+					(size 1.27 1.27)
+				)
+			)
+		)
+		(property "Datasheet" ""
+			(at 147.32 92.71 0)
+			(hide yes)
+			(show_name no)
+			(do_not_autoplace no)
+			(effects
+				(font
+					(size 1.27 1.27)
+				)
+			)
+		)
+		(property "Description" "Special symbol for telling ERC where power comes from"
+			(at 147.32 92.71 0)
+			(hide yes)
+			(show_name no)
+			(do_not_autoplace no)
+			(effects
+				(font
+					(size 1.27 1.27)
+				)
+			)
+		)
+		(pin "1"
+		)
+		(instances
+			(project "zasilacz_projekt_kompetencyjny"
+				(path "/e9ad3936-200e-4b7c-85fb-533ca6ea54fd/38eb48c3-6dca-4780-b12d-acca55a9d974"
+					(reference "#FLG02")
+					(unit 1)
+				)

Commit message: dodanie wentylatora, drobne zmiany wartości elementów
Parts:
- R3: value 0.214 -> 0.33
- U5: footprint Package_TO_SOT_SMD:SOT-223-3_TabPin2 -> Package_TO_SOT_SMD:TO-252-2
Changed lines of the file:
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@@
 			)
 		)
-		(property "Footprint" "Package_TO_SOT_SMD:SOT-223-3_TabPin2"
+		(property "Footprint" "Package_TO_SOT_SMD:TO-252-2"
 			(at 161.29 87.63 0)
 			(hide yes)
@@
 			)
 		)
-		(property "Value" "0.214"
+		(property "Value" "0.33"
 			(at 100.33 41.91 90)
 			(show_name no)
