File: main_buck.kicad_sch (KiCad schematic)
At the start: 24 parts, among them Q1 FQP30N06L, Q2 FQP30N06L, U1 IR2109, U4 LM317_TO-263, U8 LDI75L12UA

Commit message: dodanie pcb vin
Parts:
- C6: footprint Capacitor_SMD:CP_Elec_18x17.5 -> Capacitor_THT:CP_Radial_D10.0mm_P5.00mm
Changed lines of the file:
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@@
 			)
 		)
-		(property "Footprint" "Capacitor_SMD:CP_Elec_18x17.5"
+		(property "Footprint" "Capacitor_THT:CP_Radial_D10.0mm_P5.00mm"
 			(at 190.1952 95.25 0)
 			(hide yes)

Commit message: Pętla mocy i wyjście zasilania. Sterownik bramek tranzystorów
Parts:
- Vout_main_+1: footprint Connector_Wire:SolderWire-1.5sqmm_1x01_D1.7mm_OD3mm -> (none)
- fuze_out1: footprint (none) -> Connector_Wire:SolderWire-1.5sqmm_1x01_D1.7mm_OD3mm
Connections:
- net Vinm: no longer Vout_main_+1.1 (Pin_1)
- net Vout_main: now also Vout_main_+1.1 (Pin_1)
Other:
- moved on the sheet: Vout_main_+1
Changed lines of the file:
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@@
 	)
 	(junction
-		(at 217.17 83.82)
-		(diameter 0)
-		(color 0 0 0 0)
-	)
-	(junction
 		(at 189.23 83.82)
 		(diameter 0)
@@
 	)
 	(junction
+		(at 243.84 83.82)
+		(diameter 0)
+		(color 0 0 0 0)
+	)
+	(junction
 		(at 73.66 66.04)
 		(diameter 0)
@@
 	(wire
 		(pts
-			(xy 233.68 83.82) (xy 217.17 83.82)
-		)
-		(stroke
-			(width 0)
-			(type default)
-		)
-	)
-	(wire
-		(pts
 			(xy 39.37 66.04) (xy 44.45 66.04)
 		)
@@
 	(wire
 		(pts
+			(xy 243.84 81.28) (xy 243.84 83.82)
+		)
+		(stroke
+			(width 0)
+			(type default)
+		)
+	)
+	(wire
+		(pts
 			(xy 189.23 95.25) (xy 189.23 106.68)
 		)
@@
 	(wire
 		(pts
-			(xy 241.3 83.82) (xy 247.65 83.82)
+			(xy 241.3 83.82) (xy 243.84 83.82)
 		)
 		(stroke
@@
 	(wire
 		(pts
-			(xy 217.17 81.28) (xy 217.17 83.82)
-		)
-		(stroke
-			(width 0)
-			(type default)
-		)
-	)
-	(wire
-		(pts
 			(xy 186.69 83.82) (xy 184.15 83.82)
 		)
@@
 	(wire
 		(pts
-			(xy 210.82 83.82) (xy 217.17 83.82)
+			(xy 210.82 83.82) (xy 233.68 83.82)
 		)
 		(stroke
@@
 	(wire
 		(pts
+			(xy 243.84 83.82) (xy 247.65 83.82)
+		)
+		(stroke
+			(width 0)
+			(type default)
+		)
+	)
+	(wire
+		(pts
 			(xy 119.38 71.12) (xy 134.62 71.12)
 		)
@@
 			)
 		)
-		(property "Footprint" ""
+		(property "Footprint" "Connector_Wire:SolderWire-1.5sqmm_1x01_D1.7mm_OD3mm"
 			(at 237.49 85.598 90)
 			(hide yes)
@@
 	(symbol
 		(lib_id "Connector:Conn_01x01_Pin")
-		(at 217.17 76.2 270)
+		(at 243.84 76.2 270)
 		(unit 1)
 		(body_style 1)
@@
 		(fields_autoplaced yes)
 		(property "Reference" "Vout_main_+1"
-			(at 218.44 75.5649 90)
+			(at 245.11 75.5649 90)
 			(show_name no)
 			(do_not_autoplace no)
@@
 		)
 		(property "Value" "Conn_01x01_Pin"
-			(at 218.44 78.1049 90)
+			(at 245.11 78.1049 90)
 			(show_name no)
 			(do_not_autoplace no)
@@
 			)
 		)
-		(property "Footprint" "Connector_Wire:SolderWire-1.5sqmm_1x01_D1.7mm_OD3mm"
-			(at 217.17 76.2 0)
+		(property "Footprint" ""
+			(at 243.84 76.2 0)
 			(hide yes)
 			(show_name no)
@@
 		)
 		(property "Datasheet" ""
-			(at 217.17 76.2 0)
+			(at 243.84 76.2 0)
 			(hide yes)
 			(show_name no)
@@
 		)
 		(property "Description" "Generic connector, single row, 01x01, script generated"
-			(at 217.17 76.2 0)
+			(at 243.84 76.2 0)
 			(hide yes)
 			(show_name no)
