File: zasilacz_projekt_kompetencyjny.kicad_pcb (KiCad board)
At the start: 2 copper layers, 78 parts, among them J1 Program Connector, J2 UART, J3 LCD ILI9488, Q1 FQP30N06L, Q2 FQP30N06L, SW1 Voltage, SW2 Current, U3 MC34063AD, U4 LM317_TO-263, U5 NCP1117-3.3_SOT223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

Commit message: walidacja schematu, dodanie footprintu do drivera, ERC
Parts:
- added Csw1: 100n, Capacitor_SMD:C_0805_2012Metric_Pad1.18x1.45mm_HandSolder, F.Cu at (246.5, 88.2)
- added Csw2: 100n, Capacitor_SMD:C_0805_2012Metric_Pad1.18x1.45mm_HandSolder, F.Cu at (246.5, 91.2)
- added Rsw1: 10k, Resistor_SMD:R_0805_2012Metric_Pad1.20x1.40mm_HandSolder, F.Cu at (251.3, 88.2)
- added Rsw2: 10k, Resistor_SMD:R_0805_2012Metric_Pad1.20x1.40mm_HandSolder, F.Cu at (251.3, 91.2)
- added U1: IR2109, IR2109:SOIC127P600X175-8N, F.Cu at (248.3, 98.0)
- added Vout_main_+1: Conn_01x01_Pin, Connector_Wire:SolderWire-1.5sqmm_1x01_D1.7mm_OD3mm, F.Cu at (230.3, 144.1)
- added Vout_main_-1: Conn_01x01_Pin, Connector_Wire:SolderWire-1.5sqmm_1x01_D1.7mm_OD3mm, F.Cu at (230.3, 149.3)
- moved C10 132.4 mm to (231.5, 72.3)
- moved C13 132.4 mm to (200.6, 144.6)
- moved C14 132.4 mm to (200.6, 147.6)
- moved C2 132.4 mm to (214.5, 82.0)
- moved C3 132.4 mm to (200.6, 138.6)
- moved C4 132.4 mm to (200.6, 141.6)
- moved Cain1 132.4 mm to (229.5, 105.6)
- moved Cain2 132.4 mm to (229.5, 108.6)
- moved Cc1 132.4 mm to (229.5, 111.6)
- moved Cin1 132.4 mm to (229.5, 114.6)
- moved Cin2 132.4 mm to (229.5, 117.6)
- moved Cin3 132.4 mm to (229.5, 120.6)
- moved Cm1 132.4 mm to (229.5, 123.6)
- moved Cref1 132.4 mm to (229.5, 126.7)
- moved D1 132.4 mm to (204.8, 93.2)
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Connections:
- SW1 pad S2: Net-(U7-PA11) -> Net-(Csw1-Pad2)
- SW2 pad S2: Net-(U7-PA12) -> Net-(Csw2-Pad1)

Commit message: dodanie pcb vin
Parts:
- C6: footprint Capacitor_SMD:CP_Elec_18x17.5 -> Capacitor_THT:CP_Radial_D10.0mm_P5.00mm
- moved C10 257.4 mm to (1.01, -42.1)
- moved C11 257.4 mm to (10.1, -36.7)
- moved C12 257.4 mm to (10.1, -30.9)
- moved C13 257.4 mm to (-29.9, 30.1)
- moved C14 257.4 mm to (-29.9, 33.1)
- moved C3 257.4 mm to (-29.9, 24.1)
- moved C4 257.4 mm to (-29.9, 27.1)
- moved C5 257.4 mm to (-36.8, 33.7)
- moved C7 257.4 mm to (13.4, -54.5)
- moved C8 257.4 mm to (16.4, -38.1)
- moved C9 257.4 mm to (16.4, -35.1)
- moved Cain1 257.4 mm to (-1.05, -8.92)
- moved Cain2 257.4 mm to (-1.05, -5.91)
- moved Cc1 257.4 mm to (-1.05, -2.90)
- moved Cin1 257.4 mm to (-1.05, 0.11)
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Routing:
- net /input_power/N: track 0.00 -> 64.5 mm
- net Vin_32v: track 0.00 -> 46.0 mm
- net GND: track 0.00 -> 28.1 mm
- net Net-(L_pierwotne_trafo1-Pin_1): track 0.00 -> 17.5 mm
- net Net-(L_wtórne_trafo2-Pin_1): track 0.00 -> 11.3 mm
- net Net-(L_wtórne_trafo1-Pin_1): track 0.00 -> 10.3 mm
- net Net-(L3-Pin_1): track 0.00 -> 8.50 mm
- net /input_power/L: track 0.00 -> 7.00 mm
Other:
- board outline added: 236.1 x 110.6 mm

Commit message: Pętla mocy i wyjście zasilania. Sterownik bramek tranzystorów
Parts:
- removed Vout_main_+1: Conn_01x01_Pin, Connector_Wire:SolderWire-1.5sqmm_1x01_D1.7mm_OD3mm
- added fuze_out1: Fuse, Connector_Wire:SolderWire-1.5sqmm_1x01_D1.7mm_OD3mm, F.Cu at (234.8, 90.5)
- R_i_mesure1: moved to B.Cu
- moved Vout_main_-1 243.3 mm to (234.8, 97.8)
- moved R_i_mesure1 243.0 mm to (212.2, 97.8)
- moved TP_za_cewka1 63.9 mm to (204.8, 83.8)
- moved C2 47.4 mm to (162.8, 71.5)
- moved C6 39.3 mm to (191.9, 79.8), turned to 180 degrees
- moved RG1 36.9 mm to (173.0, 67.0), turned to 90 degrees
- moved RG2 34.2 mm to (185.5, 67.0), turned to 90 degrees
- moved U1 33.9 mm to (171.8, 83.5), turned to 90 degrees
- moved U7 25.1 mm to (35.2, -3.25)
- moved L1 15.9 mm to (217.0, 63.4)
- moved TP_przed_cewka1 14.3 mm to (204.8, 59.0)
Routing:
- net GND: track 28.1 -> 161.8 mm, vias 0 -> 1
- net Vinm: track 0.00 -> 80.0 mm
- net Net-(D4-A2): track 0.00 -> 75.1 mm
- net Vin_32v: track 46.0 -> 92.0 mm
- net OUT_GND_i_mesure: track 0.00 -> 19.4 mm
- net Net-(U1-LO): track 0.00 -> 17.9 mm
- net Net-(U1-HO): track 0.00 -> 13.6 mm
- net Net-(Q2-G): track 0.00 -> 3.85 mm
- net Net-(Q1-G): track 0.00 -> 3.85 mm

Commit message: Narysowanie części cyfrowej płytki, części zasialania przetwornicy głównej oraz zasilania części cyfrowej, do dokończenia połączenia mas oraz zasilań
Parts:
- added +wentylator1: Conn_01x01_Pin, Connector_Wire:SolderWire-1.5sqmm_1x01_D1.7mm_OD3mm, F.Cu at (155.2, 59.0)
- added -wentylator1: Conn_01x01_Pin, Connector_Wire:SolderWire-1.5sqmm_1x01_D1.7mm_OD3mm, F.Cu at (156.0, 84.0)
- added R6: 200, Resistor_THT:R_Axial_DIN0411_L9.9mm_D3.6mm_P15.24mm_Horizontal, F.Cu at (160.8, 58.4)
- C3, D4, R1, R2, U4: moved to B.Cu
- R3: value 0.214 -> 0.33
- U5: footprint Package_TO_SOT_SMD:SOT-223-3_TabPin2 -> Package_TO_SOT_SMD:TO-252-2
- moved D4 248.0 mm to (185.5, 106.2), turned to -90 degrees
- moved D3 231.9 mm to (170.5, 95.5), turned to -90 degrees
- moved C5 220.6 mm to (175.0, 95.3), turned to -90 degrees
- moved U8 217.3 mm to (165.2, 91.0), turned to 90 degrees
- moved U4 214.7 mm to (176.0, 100.2)
- moved C3 213.1 mm to (171.8, 93.0)
- moved C4 212.9 mm to (175.0, 84.8), turned to 90 degrees
- moved TP_pwm_za_r1 210.9 mm to (194.0, 105.8)
- moved C14 207.3 mm to (167.2, 97.0), turned to -90 degrees
- moved C7 204.3 mm to (149.2, 98.1), turned to 90 degrees
- moved R1 203.8 mm to (172.2, 107.8), turned to 180 degrees
- moved R2 203.5 mm to (172.2, 110.0)
- moved C13 202.2 mm to (164.2, 86.5), turned to 180 degrees
- moved Rpwmd1 197.7 mm to (183.2, 88.5), turned to 180 degrees
- moved L2 195.6 mm to (127.0, 95.0), turned to -90 degrees
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Connections:
- Rpwmd1 pad 1: GNDD -> GND
- Rpwmd1 pad 2: Net-(TP_pwm_przed_r1-Pin_1) -> PWM_IN
Routing:
- net Vinm: track 80.0 -> 254.5 mm
- net PWM_IN: track 0.00 -> 154.4 mm
- net OUT_GND_i_mesure: track 19.4 -> 156.2 mm, vias 0 -> 1
- net GND: track 161.8 -> 267.6 mm, vias 1 -> 7
- net Net-(D4-A2): track 75.1 -> 166.5 mm, vias 0 -> 3
- net Vin_32v: track 92.0 -> 177.7 mm, vias 0 -> 4
- net Net-(D4-A1): track 0.00 -> 50.1 mm, vias 0 -> 3
- net GNDD: track 0.00 -> 40.7 mm
- net Net-(U5-VI): track 0.00 -> 37.0 mm
- net Net-(Csw1-Pad2): track 0.00 -> 35.7 mm, vias 0 -> 2
- net /digital/PC_UART_TX: track 0.00 -> 35.6 mm
- net /digital/PC_UART_RX: track 0.00 -> 32.9 mm
- net 3.3V: track 0.00 -> 31.6 mm
- net Net-(U7-PB4): track 0.00 -> 30.9 mm
- net Net-(J3-Pin_4): track 0.00 -> 29.8 mm, vias 0 -> 2
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- added copper zone on B.Cu, net GND
Other:
- board size 236.1 x 110.6 mm -> 222.7 x 62.9 mm

Commit message: zakończenie projektu pcb
Parts:
- removed TP_GND1, TP_GNDD1: Conn_01x01_Pin, Connector_PinHeader_2.54mm:PinHeader_1x01_P2.54mm_Vertical
- added REF**: MountingHole_3.2mm_M3, MountingHole:MountingHole_3.2mm_M3, F.Cu at (23.5, 54.0)
- added REF**: MountingHole_3.2mm_M3, MountingHole:MountingHole_3.2mm_M3, F.Cu at (235.0, 112.0)
- added REF**: MountingHole_3.2mm_M3, MountingHole:MountingHole_3.2mm_M3, F.Cu at (235.0, 54.5)
- added REF**: MountingHole_3.2mm_M3, MountingHole:MountingHole_3.2mm_M3, F.Cu at (24.0, 112.0)
- moved jumper1 38.4 mm to (88.0, 91.0)
- moved D5 33.5 mm to (108.0, 106.0)
Routing:
- net 3.3V: track 31.6 -> 217.1 mm, vias 0 -> 4
- net GND: track 267.6 -> 385.8 mm, vias 7 -> 16
- net GNDD: track 40.7 -> 105.5 mm, vias 0 -> 1
- added copper zone on F.Cu, net GND
- added copper zone on F.Cu, net GNDD
Other:
- board size 222.7 x 62.9 mm -> 222.7 x 69.8 mm
- board text added: "MK, DG, KM, BB, WN"
- board text added: "Projekt kompetencyjny zasilacz regulowany 2026"
